Commit message: urdf package converted to ROS2, successfully built.

File: src/uam-model/urdf/uam-model.urdf (robot description, URDF)
Before this commit: robot Drone.SLDASM, 8 links, 7 joints
Links:
- link End_link: geometry collision mesh filename=package://uam-model/meshes/End_link.STL; visual mesh filename=package://uam-model/meshes/End_link.STL
- link Inter_link: geometry collision mesh filename=package://uam-model/meshes/Inter_link.STL; visual mesh filename=package://uam-model/meshes/Inter_link.STL
- link Manip_base_link: geometry collision mesh filename=package://uam-model/meshes/Manip_base_link.STL; visual mesh filename=package://uam-model/meshes/Manip_base_link.STL
- link Prop1_link: geometry collision mesh filename=package://uam-model/meshes/Prop1_link.STL; visual mesh filename=package://uam-model/meshes/Prop1_link.STL
- link Prop2_link: geometry collision mesh filename=package://uam-model/meshes/Prop2_link.STL; visual mesh filename=package://uam-model/meshes/Prop2_link.STL
- link Prop3_link: geometry collision mesh filename=package://uam-model/meshes/Prop3_link.STL; visual mesh filename=package://uam-model/meshes/Prop3_link.STL
- link Prop4_link: geometry collision mesh filename=package://uam-model/meshes/Prop4_link.STL; visual mesh filename=package://uam-model/meshes/Prop4_link.STL
- link base_link: geometry collision mesh filename=package://uam-model/meshes/base_link.STL; visual mesh filename=package://uam-model/meshes/base_link.STL
