Commit message: updates

File: src/uamv0_description/urdf/uamv0.urdf (robot description, URDF)
Before this commit: robot uam-model, 8 links, 7 joints
Links:
- link End_link: geometry collision mesh filename=package://uamv0_description/meshes/End_link.STL; visual mesh filename=package://uamv0_description/meshes/End_link.STL
- link Inter_link: geometry collision mesh filename=package://uamv0_description/meshes/Inter_link.STL; visual mesh filename=package://uamv0_description/meshes/Inter_link.STL
- link Manip_base_link: geometry collision mesh filename=package://uamv0_description/meshes/Manip_base_link.STL; visual mesh filename=package://uamv0_description/meshes/Manip_base_link.STL
- link Prop1_link: geometry collision mesh filename=package://uamv0_description/meshes/Prop1_link.STL; visual mesh filename=package://uamv0_description/meshes/Prop1_link.STL
- link Prop2_link: geometry collision mesh filename=package://uamv0_description/meshes/Prop2_link.STL; visual mesh filename=package://uamv0_description/meshes/Prop2_link.STL
- link Prop3_link: geometry collision mesh filename=package://uamv0_description/meshes/Prop3_link.STL; visual mesh filename=package://uamv0_description/meshes/Prop3_link.STL
- link Prop4_link: geometry collision mesh filename=package://uamv0_description/meshes/Prop4_link.STL; visual mesh filename=package://uamv0_description/meshes/Prop4_link.STL
- link base_link: geometry collision mesh filename=package://uamv0_description/meshes/base_link.STL; visual mesh filename=package://uamv0_description/meshes/base_link.STL
